File: midiBox3/midiBox3_b.kicad_pcb (KiCad board)
At the start: 2 copper layers, 100 x 100 mm, 127 parts, among them J1 BarrelJack, J2 DIN5 IN, J3 WaveBlaster, J4 DIN5 OUT, J5 RSA 2x, J6 STM32_PROG, J7 LED_CON, J8 USB_B_Micro, Q1 IRFL110, SW1 D_VALUE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

Commit message: New PCB
Parts:
- removed J8: USB_B_Micro, Connector_USB:USB_Micro-B_Molex_47346-0001
- removed MH1, MH2, MH3, MH4: MountingHole_3.2mm_M3, MountingHole:MountingHole_3.2mm_M3
- removed R32, R34: 10K, Resistor_SMD:R_0805_2012Metric_Pad1.15x1.40mm_HandSolder
- removed R33: 1.5K, Resistor_SMD:R_0805_2012Metric_Pad1.15x1.40mm_HandSolder
- removed the REF** at (109.5, 86.3)
- removed U3*: TRACO_TMR-1222_THT, Converter_DCDC:Converter_DCDC_TRACO_TMR-xxxx_THT
- removed USB1: VBUS, Connector_Pin:Pin_D0.7mm_L6.5mm_W1.8mm_FlatFork
- removed USB2: GND, Connector_Pin:Pin_D0.7mm_L6.5mm_W1.8mm_FlatFork
- removed USB3: D-, Connector_Pin:Pin_D0.7mm_L6.5mm_W1.8mm_FlatFork
- removed USB4: D+, Connector_Pin:Pin_D0.7mm_L6.5mm_W1.8mm_FlatFork
- added REF**: Converter_DCDC_TRACO_TMR-xxxx_THT, Converter_DCDC:Converter_DCDC_TRACO_TMR-xxxx_THT, F.Cu at (112.0, 47.9)
- Y1: value Crystal_GND24 -> 16MHz
- moved C36 63.2 mm to (123.3, 73.1), turned to 0 degrees
- moved U7 41.8 mm to (121.4, 79.1), turned to 0 degrees
- moved R2 39.2 mm to (112.2, 26.4)
- moved R16 34.5 mm to (113.4, 82.3), turned to 0 degrees
- moved R23 33.2 mm to (113.4, 80.3), turned to 0 degrees
- moved R20 30.8 mm to (113.4, 75.8), turned to 0 degrees
- moved R19 28.1 mm to (113.4, 77.8), turned to 0 degrees
- moved C1 20.3 mm to (63.0, 78.0), turned to 270 degrees
- moved R18 19.0 mm to (85.6, 104.7), turned to 270 degrees
- moved C30 18.1 mm to (98.8, 89.2), turned to 180 degrees
- moved C29 16.4 mm to (88.0, 87.5)
- moved R24 15.7 mm to (54.5, 115.0)
- moved C24 15.5 mm to (75.3, 97.8)
- moved C23 15.1 mm to (75.3, 91.8)
- moved R21 14.6 mm to (86.0, 100.0), turned to 180 degrees
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Connections:
- J1 pad 3: Net-(J1-Pad3) -> (no net)
- J2 pad 1: Net-(J2-Pad1) -> (no net)
- J2 pad 2: Net-(J2-Pad2) -> (no net)
- J2 pad 3: Net-(J2-Pad3) -> (no net)
- J3 pad 1: Net-(J3-Pad1) -> (no net)
- J3 pad 11: Net-(J3-Pad11) -> (no net)
- J3 pad 14: Net-(J3-Pad14) -> (no net)
- J3 pad 15: Net-(J3-Pad15) -> (no net)
- J3 pad 7: Net-(J3-Pad7) -> (no net)
- J4 pad 1: Net-(J4-Pad1) -> (no net)
- J4 pad 3: Net-(J4-Pad3) -> (no net)
- J6 pad 11: Net-(J6-Pad11) -> (no net)
- J6 pad 17: Net-(J6-Pad17) -> (no net)
- U2 pad 3: Net-(U2-Pad3) -> (no net)
- U6 pad 10: Net-(U6-Pad10) -> (no net)
- U6 pad 11: Net-(U6-Pad11) -> (no net)
- U6 pad 16: Net-(U6-Pad16) -> (no net)
- U6 pad 17: Net-(U6-Pad17) -> (no net)
- U6 pad 2: Net-(U6-Pad2) -> (no net)
- U6 pad 28: Net-(R33-Pad1) -> (no net)
- U6 pad 29: Net-(R32-Pad2) -> (no net)
- U6 pad 3: Net-(U6-Pad3) -> (no net)
- U6 pad 32: /D- -> (no net)
- U6 pad 33: /D+ -> (no net)
- U6 pad 4: Net-(U6-Pad4) -> (no net)
- U6 pad 43: Net-(U6-Pad43) -> (no net)
- U6 pad 45: Net-(U6-Pad45) -> (no net)
- U6 pad 46: Net-(U6-Pad46) -> (no net)
- U7 pad 10: Net-(U7-Pad10) -> (no net)
- U7 pad 12: Net-(U1-Pad12) -> (no net)
- U7 pad 13: /TX1 -> GNDD
- U7 pad 3: GNDD -> /TX1
- U7 pad 4: Net-(U7-Pad4) -> Net-(U1-Pad12)
- U7 pad 6: Net-(U7-Pad6) -> (no net)
- U7 pad 8: Net-(U7-Pad8) -> (no net)
Routing:
- net +5V: track 409.2 -> 512.7 mm, vias 1 -> 2
- net Net-(U1-Pad12): track 18.4 -> 76.6 mm, vias 0 -> 2
- net /D+: track 56.3 -> 0.00 mm, vias 4 -> 0
- net /D-: track 54.4 -> 0.00 mm, vias 4 -> 0
- net Net-(U1-Pad4): track 9.14 -> 61.5 mm
- net Net-(R18-Pad1): track 53.5 -> 8.07 mm, vias 2 -> 0
- net Net-(R32-Pad2): track 43.9 -> 0.00 mm, vias 2 -> 0
- net Net-(J4-Pad4): track 168.8 -> 128.4 mm, vias 4 -> 2
- net /MIDI_WB_CON: track 11.0 -> 48.9 mm, vias 0 -> 4
- net +3V3: track 212.9 -> 178.4 mm, vias 6 -> 5
- net /~RESET: track 70.5 -> 41.8 mm, vias 2 -> 4
- net Net-(R33-Pad1): track 21.6 -> 0.00 mm, vias 2 -> 0
- net /ENC_A: track 72.4 -> 93.5 mm, vias 0 -> 2
- net /ENC_B: track 67.2 -> 87.0 mm, vias 0 -> 2
- net -12V: track 73.3 -> 92.8 mm, vias 0 -> 2
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Other:
- board text added: "4x1K"
